File: hardware/hardware/zigbeeCape/BeagleBone_Headers.sch (KiCad schematic (older format))
At the start: 0 parts

Commit message: Added I2C pins, added signal wires to zigbee micro, fixed reset pin error
Parts:
- added U?: BeagleBone_P8, symbol BeagleBone:BeagleBone_P8
- added U?: BeagleBone_P9, symbol BeagleBone:BeagleBone_P9
Changed lines of the file:
@@
 $Descr A4 11693 8268
 encoding utf-8
-Sheet 1 3
+Sheet 3 3
 Title ""
 Date ""
@@
 Comment4 ""
 $EndDescr
+$Comp
+L BeagleBone:BeagleBone_P8 U?
+U 1 1 609FD186
+P 3600 4300
+F 0 "U?" H 3600 7065 50  0000 C CNN
+F 1 "BeagleBone_P8" H 3600 6974 50  0000 C CNN
+F 2 "" H 4200 7050 50  0001 C CNN
+F 3 "" H 4200 7050 50  0001 C CNN
+	1    3600 4300
+	1    0    0    -1
+$EndComp
+$Comp
+L BeagleBone:BeagleBone_P9 U?
+U 1 1 609FDC70
+P 7500 4350
+F 0 "U?" H 7500 7115 50  0000 C CNN
+F 1 "BeagleBone_P9" H 7500 7024 50  0000 C CNN
+F 2 "" H 7000 7000 50  0001 C CNN
+F 3 "" H 7000 7000 50  0001 C CNN
+	1    7500 4350
+	1    0    0    -1
+$EndComp
 $EndSCHEMATC
