File: hardware/hardware/zigbeeCape/zigbeeCape.sch (KiCad schematic (older format))
At the start: 48 parts

Commit message: Added beaglebone header heiarcy pins
Other:
- note added: "No. VDDR_RF is 1.8v from DCDC_SW. VDDR is 3.3v"
Changed lines of the file:
@@
 Wire Wire Line
 	9600 4850 9200 4850
+Text Notes 2900 2550 0    50   ~ 0
+No. VDDR_RF is 1.8v from DCDC_SW. VDDR is 3.3v
 $EndSCHEMATC

Commit message: Assigned Pin types, cleaned stuff up, Fixed most errors from the DRC (questions on the last few)
Parts:
- added C11: 22uF, symbol Device:C
- added C13, C16: 0.1uF, symbol Device:C
- added L1: 6.8uH, symbol Device:L
- added R1: R, symbol Device:R
- gave numbers to parts that had none: 47
Connections:
- net +3V3: now also R1.1; no longer C7.1
- net BeagleBone_Headers/BeagleBone_Reset: now also R1.2
- net DCDC_SW: now also L1.1
- net GND: now also J1.3 (GND), J1.5 (GND), C11.2, C13.2, C16.2
- net VDDR: now reaches U1.45 (VDDR)
- net VDDR: now also U1.48 (VDDR_RF), C11.1, C13.1, C16.1, L1.2
- net RESET_n: no longer names the net of J1.10 (~RESET~), R3.1, SW5.1, SW5.2, U1.35 (RESET_N)
- net RESET_n: now also C7.1
- net TCK: no longer names the net of J1.4 (SWDCLK/TCK), R7.1, U1.25 (JTAG_TCK)
- net TDI: no longer names the net of J1.8 (NC/TDI), R2.1, U1.27 (JTAG_TDI/DIO_17_HP)
- net TDO: no longer names the net of J1.6 (SWO/TDO), R4.1, U1.26 (JTAG_TDO/DIO_26_HP)
- net TMS: no longer names the net of J1.2 (SWDIO/TMS), R5.1, U1.24 (JTAG_TMS)
- no-connect marks 0 -> 12
Other:
- note added: "Main Page"
- note removed: "Can VDDR&VDDR_RF Connect to VDDs\n"
- note removed: "No. VDDR_RF is 1.8v from DCDC_SW. VDDR is 3.3v"
- moved on the sheet: C7, R3

Commit message: Fixed a few little things
Connections:
- net GND: no longer U1.46 (X48M_N), U1.47 (X48M_P), Y2.1, Y2.2
- new net: U1.46 (X48M_N), Y2.1
- new net: U1.47 (X48M_P), Y2.2
Other:
- note added: "Look for grounding with the 48MHz clk"
- note added: "Remove resistors on SPI and UART"
Changed lines of the file:
@@
 	7850 3950 7850 3850
 Wire Wire Line
-	7850 3850 7600 3850
-Wire Wire Line
-	7600 3850 7600 3500
-Wire Wire Line
 	7600 3500 7700 3500
 Wire Wire Line
@@
 Wire Wire Line
 	6600 2950 7600 2950
-Connection ~ 7600 3500
-Wire Wire Line
-	7850 3850 8100 3850
-Wire Wire Line
-	8100 3850 8100 3500
 Wire Wire Line
 	8100 3500 8000 3500
-Connection ~ 7850 3850
 Wire Wire Line
 	8100 3500 8100 2850
 Wire Wire Line
 	6600 2850 8100 2850
-Connection ~ 8100 3500
 Wire Wire Line
 	7200 3850 7200 3900
@@
 P 2850 750
 F 0 "R3" V 2643 750 50  0000 C CNN
-F 1 "DNM_10K" V 2734 750 50  0000 C CNN
+F 1 "DNM_10K" V 2750 750 50  0000 C CNN
 F 2 "" V 2780 750 50  0001 C CNN
 F 3 "~" H 2850 750 50  0001 C CNN
@@
 Wire Wire Line
 	2450 3450 2450 3500
-Text GLabel 4200 2300 0    50   Input ~ 0
+Text GLabel 4250 2350 0    50   Input ~ 0
 VDDR
 Wire Wire Line
@@
 Wire Wire Line
 	4750 2350 4750 2450
-Wire Wire Line
-	4750 2350 4650 2350
-Wire Wire Line
-	4650 2350 4650 2300
-Wire Wire Line
-	4650 2300 4200 2300
 Connection ~ 4750 2350
 $Comp
@@
 Text Notes 8450 1050 0    295  ~ 59
 Main Page
+Text Notes 8150 3450 0    39   ~ 0
+Look for grounding with the 48MHz clk
+Text Notes 6750 4400 0    39   ~ 0
+Remove resistors on SPI and UART
+Wire Wire Line
+	4250 2350 4750 2350
 $EndSCHEMATC

Commit message: Fixing Git issue
Parts:
- removed R13, R14, R15, R16, R18, R20: 10k, symbol Device:R
- removed Y2: 48MHz, symbol Device:Crystal
- added Y?: 48MHz, symbol Device:Crystal_GND24
Connections:
- net GND: now also Y?.2, Y?.4
- net at U1.46 (X48M_N): now also Y?.3
- net at U1.47 (X48M_P): now also Y?.1
Other:
- note added: "This symbol looks gross.\nMight endup changing it."
- note removed: "Look for grounding with the 48MHz clk"
- note removed: "Please Check my work on \npullup/pulldown resistors"
- note removed: "Pull up vs Pull Down on SPI clk?\nAre they needed?"
- note removed: "Purpose of DCDC_SW"
- note removed: "Remove resistors on SPI and UART"
Changed lines of the file:
@@
-$EndComp
-$Comp
-L Device:Crystal Y2
-U 1 1 607C8108
-P 7850 3500
-F 0 "Y2" H 7850 3232 50  0000 C CNN
-F 1 "48MHz" H 7850 3323 50  0000 C CNN
-F 2 "" H 7850 3500 50  0001 C CNN
-F 3 "~" H 7850 3500 50  0001 C CNN
-	1    7850 3500
-	-1   0    0    1
 $EndComp
 $Comp
@@
 $EndComp
 Wire Wire Line
-	7850 3950 7850 3850
-Wire Wire Line
-	7600 3500 7700 3500
-Wire Wire Line
 	7600 3500 7600 2950
 Wire Wire Line
 	6600 2950 7600 2950
-Wire Wire Line
-	8100 3500 8000 3500
 Wire Wire Line
 	8100 3500 8100 2850
@@
 F6 "2_4_GHZ_RF_P" I L 8000 1750 50
 $EndSheet
-Text Notes 5700 3750 0    50   ~ 0
-Purpose of DCDC_SW
 $Sheet
 S 4000 3750 800  1400
@@
 Wire Wire Line
 	3900 4200 4000 4200
-Text GLabel 6050 4900 0    50   Input ~ 0
+Text GLabel 7650 4900 0    50   Input ~ 0
 UART_RX
-Text GLabel 6000 5000 0    50   Output ~ 0
+Text GLabel 7600 5000 0    50   Output ~ 0
 UART_TX
-Text GLabel 6000 5100 0    50   Output ~ 0
+Text GLabel 7600 5100 0    50   Output ~ 0
 SPI_MISO
-Text GLabel 6000 5200 0    50   Input ~ 0
+Text GLabel 7600 5200 0    50   Input ~ 0
 SPI_MOSI
-Text GLabel 6000 5300 0    50   Input ~ 0
+Text GLabel 7600 5300 0    50   Input ~ 0
 SPI_CS
-Text GLabel 6000 5400 0    50   Input ~ 0
+Text GLabel 7600 5400 0    50   Input ~ 0
 SPI_CLK
-Text Notes 5050 4650 0    50   ~ 0
-Pull up vs Pull Down on SPI clk?\nAre they needed?
-$Comp
-L Device:R R18
-U 1 1 60B56B06
-P 7350 4700
-F 0 "R18" H 7420 4746 50  0000 L CNN
-F 1 "10k" H 7420 4655 50  0000 L CNN
-F 2 "" V 7280 4700 50  0001 C CNN
-F 3 "~" H 7350 4700 50  0001 C CNN
-	1    7350 4700
-	1    0    0    -1
-$EndComp
-$Comp
-L Device:R R16
-U 1 1 60B574AC
-P 7050 4700
-F 0 "R16" H 7120 4746 50  0000 L CNN
-F 1 "10k" H 7120 4655 50  0000 L CNN
-F 2 "" V 6980 4700 50  0001 C CNN
-F 3 "~" H 7050 4700 50  0001 C CNN
-	1    7050 4700
-	1    0    0    -1
-$EndComp
-$Comp
-L Device:R R15
-U 1 1 60B5855C
-P 6750 4700
-F 0 "R15" H 6820 4746 50  0000 L CNN
-F 1 "10k" H 6820 4655 50  0000 L CNN
-F 2 "" V 6680 4700 50  0001 C CNN
-F 3 "~" H 6750 4700 50  0001 C CNN
-	1    6750 4700
-	1    0    0    -1
-$EndComp
-$Comp
-L Device:R R14
-U 1 1 60B58776
-P 6450 4700
-F 0 "R14" H 6520 4746 50  0000 L CNN
-F 1 "10k" H 6520 4655 50  0000 L CNN
-F 2 "" V 6380 4700 50  0001 C CNN
-F 3 "~" H 6450 4700 50  0001 C CNN
-	1    6450 4700
-	1    0    0    -1
-$EndComp
-$Comp
-L power:+3.3V #PWR025
-U 1 1 60B5A5B0
-P 6450 4400
-F 0 "#PWR025" H 6450 4250 50  0001 C CNN
-F 1 "+3.3V" H 6465 4573 50  0000 C CNN
-F 2 "" H 6450 4400 50  0001 C CNN
-F 3 "" H 6450 4400 50  0001 C CNN
-	1    6450 4400
-	1    0    0    -1
-$EndComp
-Wire Wire Line
-	7650 4550 7650 4500
-Wire Wire Line
-	7650 4500 7350 4500
-Wire Wire Line
-	7350 4550 7350 4500
-Connection ~ 7350 4500
-Wire Wire Line
-	6450 4500 6450 4400
-Wire Wire Line
-	6450 4500 6750 4500
-Wire Wire Line
-	6450 4500 6450 4550
-Connection ~ 6450 4500
-Wire Wire Line
-	6750 4550 6750 4500
-Connection ~ 6750 4500
-Wire Wire Line
-	6750 4500 7050 4500
-Wire Wire Line
-	7050 4550 7050 4500
-Connection ~ 7050 4500
-Wire Wire Line
-	7050 4500 7350 4500
-Wire Wire Line
-	7650 4850 7650 4900
-Wire Wire Line
-	7650 4900 7850 4900
-Connection ~ 7650 4900
-Wire Wire Line
-	7850 5000 7350 5000
-Wire Wire Line
-	7850 5200 6750 5200
-Wire Wire Line
-	7850 5300 6450 5300
-Wire Wire Line
-	7350 4850 7350 5000
-Connection ~ 7350 5000
-Wire Wire Line
-	7050 4850 7050 5100
-Connection ~ 7050 5100
-Wire Wire Line
-	7050 5100 7850 5100
-Wire Wire Line
-	6750 4850 6750 5200
-Connection ~ 6750 5200
-Wire Wire Line
-	6450 4850 6450 5300
-Connection ~ 6450 5300
-$Comp
-L Device:R R13
-U 1 1 60C3C131
-P 6150 5650
-F 0 "R13" H 6220 5696 50  0000 L CNN
-F 1 "10k" H 6220 5605 50  0000 L CNN
-F 2 "" V 6080 5650 50  0001 C CNN
-F 3 "~" H 6150 5650 50  0001 C CNN
-	1    6150 5650
-	1    0    0    -1
-$EndComp
-Wire Wire Line
-	6000 5300 6450 5300
-Wire Wire Line
-	6000 5200 6750 5200
-Wire Wire Line
-	6000 5100 7050 5100
-Wire Wire Line
-	6000 5000 7350 5000
-Wire Wire Line
-	6050 4900 7650 4900
-Wire Wire Line
-	6000 5400 6150 5400
-Wire Wire Line
-	6150 5500 6150 5400
-Connection ~ 6150 5400
-Wire Wire Line
-	6150 5400 7850 5400
-$Comp
-L power:GND #PWR023
-U 1 1 60CB9CE2
-P 6150 5900
-F 0 "#PWR023" H 6150 5650 50  0001 C CNN
-F 1 "GND" H 6155 5727 50  0000 C CNN
-F 2 "" H 6150 5900 50  0001 C CNN
-F 3 "" H 6150 5900 50  0001 C CNN
-	1    6150 5900
-	1    0    0    -1
-$EndComp
-Wire Wire Line
-	6150 5800 6150 5900
 Text Notes 2900 3400 0    50   ~ 0
 Place capacitors close to refered pin. 22uf and 0.1uf on pin 34
@@
 Wire Wire Line
 	4000 4900 3900 4900
-$Comp
-L Device:R R20
-U 1 1 60B56235
-P 7650 4700
-F 0 "R20" H 7720 4746 50  0000 L CNN
-F 1 "10k" H 7720 4655 50  0000 L CNN
-F 2 "" V 7580 4700 50  0001 C CNN
-F 3 "~" H 7650 4700 50  0001 C CNN
-	1    7650 4700
-	1    0    0    -1
-$EndComp
-Text Notes 5050 4450 0    50   ~ 0
-Please Check my work on \npullup/pulldown resistors
 $Comp
 L Device:R R19
@@
 Text Notes 8450 1050 0    295  ~ 59
 Main Page
-Text Notes 8150 3450 0    39   ~ 0
-Look for grounding with the 48MHz clk
-Text Notes 6750 4400 0    39   ~ 0
-Remove resistors on SPI and UART
 Wire Wire Line
 	4250 2350 4750 2350
+$Comp
+L Device:Crystal_GND24 Y?
+U 1 1 60907ED1
+P 7850 3500
+F 0 "Y?" H 8044 3546 50  0000 L CNN
+F 1 "48MHz" H 8044 3455 50  0000 L CNN
+F 2 "" H 7850 3500 50  0001 C CNN
+F 3 "~" H 7850 3500 50  0001 C CNN
+	1    7850 3500
+	1    0    0    -1
+$EndComp
+Wire Wire Line
+	7600 3500 7700 3500
+Wire Wire Line
+	8000 3500 8100 3500
+Wire Wire Line
+	7850 3300 7850 3200
+Wire Wire Line
+	7850 3200 8300 3200
+Wire Wire Line
+	8300 3200 8300 3750
+Wire Wire Line
+	8300 3750 7850 3750
+Wire Wire Line
+	7850 3750 7850 3950
+Wire Wire Line
+	7850 3750 7850 3700
+Connection ~ 7850 3750
+Wire Wire Line
+	7650 4900 7850 4900
+Wire Wire Line
+	7850 5000 7600 5000
+Wire Wire Line
+	7600 5100 7850 5100
+Wire Wire Line
+	7850 5200 7600 5200
+Wire Wire Line
+	7600 5300 7850 5300
+Wire Wire Line
+	7850 5400 7600 5400
+Text Notes 8200 3100 0    39   ~ 0
+This symbol looks gross.\nMight endup changing it.
 $EndSCHEMATC

Commit message: Started BOM
Parts:
- gave numbers to parts that had none: 1
Changed lines of the file:
@@
 	4250 2350 4750 2350
 $Comp
-L Device:Crystal_GND24 Y?
+L Device:Crystal_GND24 Y2
 U 1 1 60907ED1
 P 7850 3500
-F 0 "Y?" H 8044 3546 50  0000 L CNN
+F 0 "Y2" H 8044 3546 50  0000 L CNN
 F 1 "48MHz" H 8044 3455 50  0000 L CNN
 F 2 "" H 7850 3500 50  0001 C CNN

Commit message: Added excell file to document deviations from CC1352R1 footprint size. Started assigning Footprints for Zigbee cape
Parts:
- C1, C10, C2, C3, C4, C5, C6, C7, C8, C9: footprint (none) -> Capacitor_SMD:C_0603_1608Metric_Pad1.08x0.95mm_HandSolder
Changed lines of the file:
@@
 F 0 "C1" H 1765 5946 50  0000 L CNN
 F 1 "DNM_1uF" H 1765 5855 50  0000 L CNN
-F 2 "" H 1688 5750 50  0001 C CNN
+F 2 "Capacitor_SMD:C_0603_1608Metric_Pad1.08x0.95mm_HandSolder" H 1688 5750 50  0001 C CNN
 F 3 "~" H 1650 5900 50  0001 C CNN
 	1    1650 5900
@@
 F 0 "C2" H 1765 6646 50  0000 L CNN
 F 1 "DNM_1uF" H 1765 6555 50  0000 L CNN
-F 2 "" H 1688 6450 50  0001 C CNN
+F 2 "Capacitor_SMD:C_0603_1608Metric_Pad1.08x0.95mm_HandSolder" H 1688 6450 50  0001 C CNN
 F 3 "~" H 1650 6600 50  0001 C CNN
 	1    1650 6600
@@
 F 0 "C3" H 1765 7346 50  0000 L CNN
 F 1 "DNM_1uF" H 1765 7255 50  0000 L CNN
-F 2 "" H 1688 7150 50  0001 C CNN
+F 2 "Capacitor_SMD:C_0603_1608Metric_Pad1.08x0.95mm_HandSolder" H 1688 7150 50  0001 C CNN
 F 3 "~" H 1650 7300 50  0001 C CNN
 	1    1650 7300
@@
 F 0 "C10" H 4565 2996 50  0000 L CNN
 F 1 "22uF" H 4565 2905 50  0000 L CNN
-F 2 "" H 4488 2800 50  0001 C CNN
+F 2 "Capacitor_SMD:C_0603_1608Metric_Pad1.08x0.95mm_HandSolder" H 4488 2800 50  0001 C CNN
 F 3 "~" H 4450 2950 50  0001 C CNN
 	1    4450 2950
@@
 F 0 "C9" H 4115 2996 50  0000 L CNN
 F 1 "0.1uF" H 4115 2905 50  0000 L CNN
-F 2 "" H 4038 2800 50  0001 C CNN
+F 2 "Capacitor_SMD:C_0603_1608Metric_Pad1.08x0.95mm_HandSolder" H 4038 2800 50  0001 C CNN
 F 3 "~" H 4000 2950 50  0001 C CNN
 	1    4000 2950
@@
 F 0 "C8" H 3665 2996 50  0000 L CNN
 F 1 "0.1uF" H 3665 2905 50  0000 L CNN
-F 2 "" H 3588 2800 50  0001 C CNN
+F 2 "Capacitor_SMD:C_0603_1608Metric_Pad1.08x0.95mm_HandSolder" H 3588 2800 50  0001 C CNN
 F 3 "~" H 3550 2950 50  0001 C CNN
 	1    3550 2950
@@
 F 0 "C6" H 3215 2996 50  0000 L CNN
 F 1 "0.1uF" H 3215 2905 50  0000 L CNN
-F 2 "" H 3138 2800 50  0001 C CNN
+F 2 "Capacitor_SMD:C_0603_1608Metric_Pad1.08x0.95mm_HandSolder" H 3138 2800 50  0001 C CNN
 F 3 "~" H 3100 2950 50  0001 C CNN
 	1    3100 2950
@@
 F 0 "C5" H 2765 2996 50  0000 L CNN
 F 1 "0.1uF" H 2765 2905 50  0000 L CNN
-F 2 "" H 2688 2800 50  0001 C CNN
+F 2 "Capacitor_SMD:C_0603_1608Metric_Pad1.08x0.95mm_HandSolder" H 2688 2800 50  0001 C CNN
 F 3 "~" H 2650 2950 50  0001 C CNN
 	1    2650 2950
@@
 F 0 "C4" H 2715 4096 50  0000 L CNN
 F 1 "DNM_2.2uF" H 2715 4005 50  0000 L CNN
-F 2 "" H 2638 3900 50  0001 C CNN
+F 2 "Capacitor_SMD:C_0603_1608Metric_Pad1.08x0.95mm_HandSolder" H 2638 3900 50  0001 C CNN
 F 3 "~" H 2600 4050 50  0001 C CNN
 	1    2600 4050
@@
 F 0 "C7" H 3415 996 50  0000 L CNN
 F 1 "2.2uF" H 3415 905 50  0000 L CNN
-F 2 "" H 3338 800 50  0001 C CNN
+F 2 "Capacitor_SMD:C_0603_1608Metric_Pad1.08x0.95mm_HandSolder" H 3338 800 50  0001 C CNN
 F 3 "~" H 3300 950 50  0001 C CNN
 	1    3300 950

Commit message: Added items to BOM. Added footprints to GIT. Finished Capacitor footprint association. Finished LED footprint association.
Parts:
- C11, C12, C13, C14, C15, C16: footprint (none) -> Capacitor_SMD:C_0603_1608Metric_Pad1.08x0.95mm_HandSolder
- D1, D2, D3, D4, D5, D6: footprint (none) -> LED_SMD:LED_0603_1608Metric_Pad1.05x0.95mm_HandSolder
Changed lines of the file:
@@
 F 0 "D6" V 5039 6682 50  0000 R CNN
 F 1 "Green" V 4948 6682 50  0000 R CNN
-F 2 "" H 5000 6800 50  0001 C CNN
+F 2 "LED_SMD:LED_0603_1608Metric_Pad1.05x0.95mm_HandSolder" H 5000 6800 50  0001 C CNN
 F 3 "~" H 5000 6800 50  0001 C CNN
 	1    5000 6800
@@
 F 0 "D4" V 4339 6682 50  0000 R CNN
 F 1 "Blue" V 4248 6682 50  0000 R CNN
-F 2 "" H 4300 6800 50  0001 C CNN
+F 2 "LED_SMD:LED_0603_1608Metric_Pad1.05x0.95mm_HandSolder" H 4300 6800 50  0001 C CNN
 F 3 "~" H 4300 6800 50  0001 C CNN
 	1    4300 6800
@@
 F 0 "D3" V 3989 6682 50  0000 R CNN
 F 1 "Blue" V 3898 6682 50  0000 R CNN
-F 2 "" H 3950 6800 50  0001 C CNN
+F 2 "LED_SMD:LED_0603_1608Metric_Pad1.05x0.95mm_HandSolder" H 3950 6800 50  0001 C CNN
 F 3 "~" H 3950 6800 50  0001 C CNN
 	1    3950 6800
@@
 F 0 "D2" V 3639 6682 50  0000 R CNN
 F 1 "Blue" V 3548 6682 50  0000 R CNN
-F 2 "" H 3600 6800 50  0001 C CNN
+F 2 "LED_SMD:LED_0603_1608Metric_Pad1.05x0.95mm_HandSolder" H 3600 6800 50  0001 C CNN
 F 3 "~" H 3600 6800 50  0001 C CNN
 	1    3600 6800
@@
 F 0 "D5" V 4689 6682 50  0000 R CNN
 F 1 "Blue" V 4598 6682 50  0000 R CNN
-F 2 "" H 4650 6800 50  0001 C CNN
+F 2 "LED_SMD:LED_0603_1608Metric_Pad1.05x0.95mm_HandSolder" H 4650 6800 50  0001 C CNN
 F 3 "~" H 4650 6800 50  0001 C CNN
 	1    4650 6800
@@
 F 0 "D1" V 3289 6682 50  0000 R CNN
 F 1 "Blue" V 3198 6682 50  0000 R CNN
-F 2 "" H 3250 6800 50  0001 C CNN
+F 2 "LED_SMD:LED_0603_1608Metric_Pad1.05x0.95mm_HandSolder" H 3250 6800 50  0001 C CNN
 F 3 "~" H 3250 6800 50  0001 C CNN
 	1    3250 6800
@@
 F 0 "C12" H 6815 3746 50  0000 L CNN
 F 1 "12pF" H 6815 3655 50  0000 L CNN
-F 2 "" H 6738 3550 50  0001 C CNN
+F 2 "Capacitor_SMD:C_0603_1608Metric_Pad1.08x0.95mm_HandSolder" H 6738 3550 50  0001 C CNN
 F 3 "~" H 6700 3700 50  0001 C CNN
 	1    6700 3700
@@
 F 0 "C14" H 7315 3746 50  0000 L CNN
 F 1 "12pF" H 7315 3655 50  0000 L CNN
-F 2 "" H 7238 3550 50  0001 C CNN
+F 2 "Capacitor_SMD:C_0603_1608Metric_Pad1.08x0.95mm_HandSolder" H 7238 3550 50  0001 C CNN
 F 3 "~" H 7200 3700 50  0001 C CNN
 	1    7200 3700
@@
 F 0 "C15" H 7415 2496 50  0000 L CNN
 F 1 "1uF" H 7415 2405 50  0000 L CNN
-F 2 "" H 7338 2300 50  0001 C CNN
+F 2 "Capacitor_SMD:C_0603_1608Metric_Pad1.08x0.95mm_HandSolder" H 7338 2300 50  0001 C CNN
 F 3 "~" H 7300 2450 50  0001 C CNN
 	1    7300 2450
@@
 F 0 "C13" H 7015 1196 50  0000 L CNN
 F 1 "0.1uF" H 7015 1105 50  0000 L CNN
-F 2 "" H 6938 1000 50  0001 C CNN
+F 2 "Capacitor_SMD:C_0603_1608Metric_Pad1.08x0.95mm_HandSolder" H 6938 1000 50  0001 C CNN
 F 3 "~" H 6900 1150 50  0001 C CNN
 	1    6900 1150
@@
 F 0 "C11" H 6365 1196 50  0000 L CNN
 F 1 "22uF" H 6365 1105 50  0000 L CNN
-F 2 "" H 6288 1000 50  0001 C CNN
+F 2 "Capacitor_SMD:C_0603_1608Metric_Pad1.08x0.95mm_HandSolder" H 6288 1000 50  0001 C CNN
 F 3 "~" H 6250 1150 50  0001 C CNN
 	1    6250 1150
@@
 F 0 "C16" H 7465 1196 50  0000 L CNN
 F 1 "0.1uF" H 7465 1105 50  0000 L CNN
-F 2 "" H 7388 1000 50  0001 C CNN
+F 2 "Capacitor_SMD:C_0603_1608Metric_Pad1.08x0.95mm_HandSolder" H 7388 1000 50  0001 C CNN
 F 3 "~" H 7350 1150 50  0001 C CNN
 	1    7350 1150
