File: hardware/hardware/zigbeeCape/zigbeeCape.sch (KiCad schematic (older format))
At the start: 46 parts, among them J1 Conn_ARM_JTAG_SWD_10, SW1 SW_MEC_5E, SW2 SW_MEC_5E, SW3 SW_MEC_5E, SW4 SW_MEC_5E, SW5 SW_MEC_5E, U1 CC1352R, Y1 32.768kHz, Y2 48MHz

Commit message: Completed BOM except unlabled DNM parts, labled in red. Completed footprint association except onboard antenae
Parts:
- J1: footprint (none) -> zigbeeCape:Conn_ARM_JTAG_SWD_10
- L1: footprint (none) -> Inductor_SMD:L_0805_2012Metric_Pad1.15x1.40mm_HandSolder
- R1, R10, R11, R12, R17, R19, R2, R3, R4, R5, R6, R7, R8, R9: footprint (none) -> Resistor_SMD:R_0603_1608Metric_Pad0.98x0.95mm_HandSolder
- SW1, SW2, SW3, SW4, SW5: footprint (none) -> Button_Switch_THT:SW_PUSH_6mm
- U1: footprint (none) -> zigbeeCape:CC1352R
- Y1: footprint (none) -> zigbeeCape:FC-135_Crystal_Unit
- Y2: footprint (none) -> zigbeeCape:SXT32418FD16-48MHZ_Crystal
Changed lines of the file:
@@
 F 0 "U1" H 8525 6565 50  0000 C CNN
 F 1 "CC1352R" H 8525 6474 50  0000 C CNN
-F 2 "" H 8900 6750 50  0001 C CNN
+F 2 "zigbeeCape:CC1352R" H 8900 6750 50  0001 C CNN
 F 3 "" H 8900 6750 50  0001 C CNN
 	2    8300 5550
@@
 F 0 "U1" H 5700 3515 50  0000 C CNN
 F 1 "CC1352R" H 5700 3424 50  0000 C CNN
-F 2 "" H 5850 3700 50  0001 C CNN
+F 2 "zigbeeCape:CC1352R" H 5850 3700 50  0001 C CNN
 F 3 "" H 5850 3700 50  0001 C CNN
 	1    5250 2500
@@
 F 0 "SW1" H 1100 6185 50  0000 C CNN
 F 1 "SW_MEC_5E" H 1100 6094 50  0000 C CNN
-F 2 "" H 1100 6100 50  0001 C CNN
+F 2 "Button_Switch_THT:SW_PUSH_6mm" H 1100 6100 50  0001 C CNN
 F 3 "http://www.apem.com/int/index.php?controller=attachment&id_attachment=1371" H 1100 6100 50  0001 C CNN
 	1    1100 5800
@@
 F 0 "R8" H 3670 7246 50  0000 L CNN
 F 1 "1k" H 3670 7155 50  0000 L CNN
-F 2 "" V 3530 7200 50  0001 C CNN
+F 2 "Resistor_SMD:R_0603_1608Metric_Pad0.98x0.95mm_HandSolder" V 3530 7200 50  0001 C CNN
 F 3 "~" H 3600 7200 50  0001 C CNN
 	1    3600 7200
@@
 F 0 "R9" H 4020 7246 50  0000 L CNN
 F 1 "1k" H 4020 7155 50  0000 L CNN
-F 2 "" V 3880 7200 50  0001 C CNN
+F 2 "Resistor_SMD:R_0603_1608Metric_Pad0.98x0.95mm_HandSolder" V 3880 7200 50  0001 C CNN
 F 3 "~" H 3950 7200 50  0001 C CNN
 	1    3950 7200
@@
 F 0 "R10" H 4370 7246 50  0000 L CNN
 F 1 "1k" H 4370 7155 50  0000 L CNN
-F 2 "" V 4230 7200 50  0001 C CNN
+F 2 "Resistor_SMD:R_0603_1608Metric_Pad0.98x0.95mm_HandSolder" V 4230 7200 50  0001 C CNN
 F 3 "~" H 4300 7200 50  0001 C CNN
 	1    4300 7200
@@
 F 0 "R11" H 4720 7246 50  0000 L CNN
 F 1 "1k" H 4720 7155 50  0000 L CNN
-F 2 "" V 4580 7200 50  0001 C CNN
+F 2 "Resistor_SMD:R_0603_1608Metric_Pad0.98x0.95mm_HandSolder" V 4580 7200 50  0001 C CNN
 F 3 "~" H 4650 7200 50  0001 C CNN
 	1    4650 7200
@@
 F 0 "R12" H 5070 7246 50  0000 L CNN
 F 1 "1k" H 5070 7155 50  0000 L CNN
-F 2 "" V 4930 7200 50  0001 C CNN
+F 2 "Resistor_SMD:R_0603_1608Metric_Pad0.98x0.95mm_HandSolder" V 4930 7200 50  0001 C CNN
 F 3 "~" H 5000 7200 50  0001 C CNN
 	1    5000 7200
@@
 F 0 "SW2" H 1100 6885 50  0000 C CNN
 F 1 "SW_MEC_5E" H 1100 6794 50  0000 C CNN
-F 2 "" H 1100 6800 50  0001 C CNN
+F 2 "Button_Switch_THT:SW_PUSH_6mm" H 1100 6800 50  0001 C CNN
 F 3 "http://www.apem.com/int/index.php?controller=attachment&id_attachment=1371" H 1100 6800 50  0001 C CNN
 	1    1100 6500
@@
 F 0 "SW3" H 1100 7585 50  0000 C CNN
 F 1 "SW_MEC_5E" H 1100 7494 50  0000 C CNN
-F 2 "" H 1100 7500 50  0001 C CNN
+F 2 "Button_Switch_THT:SW_PUSH_6mm" H 1100 7500 50  0001 C CNN
 F 3 "http://www.apem.com/int/index.php?controller=attachment&id_attachment=1371" H 1100 7500 50  0001 C CNN
 	1    1100 7200
@@
 F 0 "R6" H 3320 7246 50  0000 L CNN
 F 1 "1k" H 3320 7155 50  0000 L CNN
-F 2 "" V 3180 7200 50  0001 C CNN
+F 2 "Resistor_SMD:R_0603_1608Metric_Pad0.98x0.95mm_HandSolder" V 3180 7200 50  0001 C CNN
 F 3 "~" H 3250 7200 50  0001 C CNN
 	1    3250 7200
@@
 F 0 "Y1" H 6950 3768 50  0000 C CNN
 F 1 "32.768kHz" H 6950 3677 50  0000 C CNN
-F 2 "" H 6950 3500 50  0001 C CNN
+F 2 "zigbeeCape:FC-135_Crystal_Unit" H 6950 3500 50  0001 C CNN
 F 3 "~" H 6950 3500 50  0001 C CNN
 	1    6950 3500
@@
 F 0 "R2" H 2670 1896 50  0000 L CNN
 F 1 "10K" H 2670 1805 50  0000 L CNN
-F 2 "" V 2530 1850 50  0001 C CNN
+F 2 "Resistor_SMD:R_0603_1608Metric_Pad0.98x0.95mm_HandSolder" V 2530 1850 50  0001 C CNN
 F 3 "~" H 2600 1850 50  0001 C CNN
 	1    2600 1850
@@
 F 0 "R4" H 2970 1896 50  0000 L CNN
 F 1 "10K" H 2970 1805 50  0000 L CNN
-F 2 "" V 2830 1850 50  0001 C CNN
+F 2 "Resistor_SMD:R_0603_1608Metric_Pad0.98x0.95mm_HandSolder" V 2830 1850 50  0001 C CNN
 F 3 "~" H 2900 1850 50  0001 C CNN
 	1    2900 1850
@@
 F 0 "R5" H 3270 1896 50  0000 L CNN
 F 1 "10K" H 3270 1805 50  0000 L CNN
-F 2 "" V 3130 1850 50  0001 C CNN
+F 2 "Resistor_SMD:R_0603_1608Metric_Pad0.98x0.95mm_HandSolder" V 3130 1850 50  0001 C CNN
 F 3 "~" H 3200 1850 50  0001 C CNN
 	1    3200 1850
@@
 F 0 "R7" H 3570 1896 50  0000 L CNN
 F 1 "10K" H 3570 1805 50  0000 L CNN
-F 2 "" V 3430 1850 50  0001 C CNN
+F 2 "Resistor_SMD:R_0603_1608Metric_Pad0.98x0.95mm_HandSolder" V 3430 1850 50  0001 C CNN
 F 3 "~" H 3500 1850 50  0001 C CNN
 	1    3500 1850
@@
 F 0 "R3" V 2643 750 50  0000 C CNN
 F 1 "DNM_10K" V 2750 750 50  0000 C CNN
-F 2 "" V 2780 750 50  0001 C CNN
+F 2 "Resistor_SMD:R_0603_1608Metric_Pad0.98x0.95mm_HandSolder" V 2780 750 50  0001 C CNN
 F 3 "~" H 2850 750 50  0001 C CNN
 	1    2850 750
@@
 F 0 "SW5" H 4150 1285 50  0000 C CNN
 F 1 "SW_MEC_5E" H 4150 1194 50  0000 C CNN
-F 2 "" H 4150 1200 50  0001 C CNN
+F 2 "Button_Switch_THT:SW_PUSH_6mm" H 4150 1200 50  0001 C CNN
 F 3 "http://www.apem.com/int/index.php?controller=attachment&id_attachment=1371" H 4150 1200 50  0001 C CNN
 	1    4150 900
@@
 F 0 "SW4" H 2050 4335 50  0000 C CNN
 F 1 "SW_MEC_5E" H 2050 4244 50  0000 C CNN
-F 2 "" H 2050 4250 50  0001 C CNN
+F 2 "Button_Switch_THT:SW_PUSH_6mm" H 2050 4250 50  0001 C CNN
 F 3 "http://www.apem.com/int/index.php?controller=attachment&id_attachment=1371" H 2050 4250 50  0001 C CNN
 	1    2050 3950
@@
 F 0 "R19" H 7620 5796 50  0000 L CNN
 F 1 "4.7k" H 7620 5705 50  0000 L CNN
-F 2 "" V 7480 5750 50  0001 C CNN
+F 2 "Resistor_SMD:R_0603_1608Metric_Pad0.98x0.95mm_HandSolder" V 7480 5750 50  0001 C CNN
 F 3 "~" H 7550 5750 50  0001 C CNN
 	1    7550 5750
@@
 F 0 "R17" H 7320 5796 50  0000 L CNN
 F 1 "4.7k" H 7320 5705 50  0000 L CNN
-F 2 "" V 7180 5750 50  0001 C CNN
+F 2 "Resistor_SMD:R_0603_1608Metric_Pad0.98x0.95mm_HandSolder" V 7180 5750 50  0001 C CNN
 F 3 "~" H 7250 5750 50  0001 C CNN
 	1    7250 5750
@@
 F 0 "R1" H 2520 3696 50  0000 L CNN
 F 1 "R" H 2520 3605 50  0000 L CNN
-F 2 "" V 2380 3650 50  0001 C CNN
+F 2 "Resistor_SMD:R_0603_1608Metric_Pad0.98x0.95mm_HandSolder" V 2380 3650 50  0001 C CNN
 F 3 "~" H 2450 3650 50  0001 C CNN
 	1    2450 3650
@@
 F 0 "L1" V 6140 900 50  0000 C CNN
 F 1 "6.8uH" V 6049 900 50  0000 C CNN
-F 2 "" H 5950 900 50  0001 C CNN
+F 2 "Inductor_SMD:L_0805_2012Metric_Pad1.15x1.40mm_HandSolder" H 5950 900 50  0001 C CNN
 F 3 "~" H 5950 900 50  0001 C CNN
 	1    5950 900
@@
 F 0 "J1" H 1607 1496 50  0000 R CNN
 F 1 "Conn_ARM_JTAG_SWD_10" H 1607 1405 50  0000 R CNN
-F 2 "" H 2050 1450 50  0001 C CNN
+F 2 "zigbeeCape:Conn_ARM_JTAG_SWD_10" H 2050 1450 50  0001 C CNN
 F 3 "http://infocenter.arm.com/help/topic/com.arm.doc.ddi0314h/DDI0314H_coresight_components_trm.pdf" V 1700 200 50  0001 C CNN
 	1    2050 1450
@@
 F 0 "Y2" H 8044 3546 50  0000 L CNN
 F 1 "48MHz" H 8044 3455 50  0000 L CNN
-F 2 "" H 7850 3500 50  0001 C CNN
+F 2 "zigbeeCape:SXT32418FD16-48MHZ_Crystal" H 7850 3500 50  0001 C CNN
 F 3 "~" H 7850 3500 50  0001 C CNN
 	1    7850 3500
