File: hardware/hardware/zigbeeCape/ZigBeeFiltering.sch (KiCad schematic (older format))
At the start: 27 parts, among them U2 0.8Ghz_and_2.4GHz_Filter, U3 SMA_Antenna

Commit message: Updated properties for faster BOM generation
Parts:
- C17, C26: Digikey Part Number (none) -> 490-5924-1-ND
- C18, C19: Digikey Part Number (none) -> 490-8189-1-ND
- C20: Digikey Part Number (none) -> 490-6209-1-ND
- C21: Digikey Part Number (none) -> 478-3659-1-ND
- C22, C29, C31: Digikey Part Number (none) -> 490-5922-1-ND
- C23, C24: Digikey Part Number (none) -> 490-5872-1-ND
- C25, C27, C28: Digikey Part Number (none) -> 490-5939-1-ND
- L10, L7: Digikey Part Number (none) -> 490-6569-1-ND
- L11, L9: Digikey Part Number (none) -> 490-2623-1-ND
- L12: Digikey Part Number (none) -> 490-8390-1-ND
- L2: Digikey Part Number (none) -> 490-2625-1-ND
- L3, L4: Digikey Part Number (none) -> 490-8389-1-ND
- L5, L6: Digikey Part Number (none) -> 490-2617-1-ND
- L8: Digikey Part Number (none) -> 490-2627-1-ND
- U2: Digikey Part Number (none) -> 445-174204-1-ND
- U3: Digikey Part Number (none) -> ACX1230-ND
Changed lines of the file:
@@
 F 2 "Capacitor_SMD:C_0402_1005Metric_Pad0.74x0.62mm_HandSolder" H 3438 4750 50  0001 C CNN
 F 3 "https://www.digikey.com/en/products/detail/murata-electronics/GRM1555C1H3R0CA01D/3175191?s=N4IgTCBcDaIOICUCyBGArBgwigEgZgQAZMBBQlAERAF0BfIA" H 3400 4900 50  0001 C CNN
+F 4 "490-5872-1-ND" H 3400 4900 50  0001 C CNN "Digikey Part Number"
 	1    3400 4900
 	0    -1   -1   0
@@
 F 2 "Inductor_SMD:L_0402_1005Metric_Pad0.77x0.64mm_HandSolder" H 2200 4900 50  0001 C CNN
 F 3 "https://www.digikey.com/en/products/detail/murata-electronics/LQG15HS3N9S02D/662866?s=N4IgTCBcDaIDIEUDiBGArACQMoGYByAnFgAxgAiIAugL5A" H 2200 4900 50  0001 C CNN
+F 4 "490-2617-1-ND" H 2200 4900 50  0001 C CNN "Digikey Part Number"
 	1    2200 4900
 	0    -1   -1   0
@@
 F 2 "Capacitor_SMD:C_0402_1005Metric_Pad0.74x0.62mm_HandSolder" H 3038 4100 50  0001 C CNN
 F 3 "https://www.digikey.com/en/products/detail/murata-electronics/GRM1555C1H101JA01D/3693829?s=N4IgTCBcDaIOICUCyBGArBgwigEigDCgFICChAIiALoC%2BQA" H 3000 4250 50  0001 C CNN
+F 4 "490-5922-1-ND" H 3000 4250 50  0001 C CNN "Digikey Part Number"
 	1    3000 4250
 	1    0    0    -1
@@
 F 2 "Inductor_SMD:L_0402_1005Metric_Pad0.77x0.64mm_HandSolder" H 2200 5300 50  0001 C CNN
 F 3 "https://www.digikey.com/en/products/detail/murata-electronics/LQG15HS3N9S02D/662866?s=N4IgTCBcDaIDIEUDiBGArACQMoGYByAnFgAxgAiIAugL5A" H 2200 5300 50  0001 C CNN
+F 4 "490-2617-1-ND" H 2200 5300 50  0001 C CNN "Digikey Part Number"
 	1    2200 5300
 	0    -1   -1   0
@@
 F 2 "Capacitor_SMD:C_0402_1005Metric_Pad0.74x0.62mm_HandSolder" H 4288 5350 50  0001 C CNN
 F 3 "~" H 4250 5500 50  0001 C CNN
+F 4 "490-5939-1-ND" H 4250 5500 50  0001 C CNN "Digikey Part Number"
 	1    4250 5500
 	1    0    0    -1
@@
 F 2 "Inductor_SMD:L_0402_1005Metric_Pad0.77x0.64mm_HandSolder" H 3000 4650 50  0001 C CNN
 F 3 "https://www.digikey.com/en/products/detail/murata-electronics/LQG15HS10NJ02D/662872?s=N4IgTCBcDaIDIEUDiBGArACQMooAwDkApXMAERAF0BfIA" H 3000 4650 50  0001 C CNN
+F 4 "490-2623-1-ND" H 3000 4650 50  0001 C CNN "Digikey Part Number"
 	1    3000 4650
 	1    0    0    -1
@@
 F 2 "Capacitor_SMD:C_0402_1005Metric_Pad0.74x0.62mm_HandSolder" H 4938 5350 50  0001 C CNN
 F 3 "https://www.digikey.com/en/products/detail/murata-electronics/GRM1555C1H3R6CA01D/3693850?s=N4IgTCBcDaIOICUCyBGArBgwigEgZgQDZMBBABhQBEQBdAXyA" H 4900 5500 50  0001 C CNN
+F 4 "490-5939-1-ND" H 4900 5500 50  0001 C CNN "Digikey Part Number"
 	1    4900 5500
 	1    0    0    -1
@@
 F 2 "Inductor_SMD:L_0402_1005Metric_Pad0.77x0.64mm_HandSolder" H 4550 5100 50  0001 C CNN
 F 3 "https://www.digikey.com/en/products/detail/murata-electronics/LQG15HS9N1J02D/2594223?s=N4IgTCBcDaIDIEUDiBGArACQMoE4ByKAUgAxgAiIAugL5A" H 4550 5100 50  0001 C CNN
+F 4 "490-8390-1-ND" H 4550 5100 50  0001 C CNN "Digikey Part Number"
 	1    4550 5100
 	0    -1   -1   0
@@
 F 2 "Capacitor_SMD:C_0402_1005Metric_Pad0.74x0.62mm_HandSolder" H 5238 4950 50  0001 C CNN
 F 3 "https://www.digikey.com/en/products/detail/murata-electronics/GRM1555C1H101JA01D/3693829?s=N4IgTCBcDaIOICUCyBGArBgwigEigDCgFICChAIiALoC%2BQA" H 5200 5100 50  0001 C CNN
+F 4 "490-5922-1-ND" H 5200 5100 50  0001 C CNN "Digikey Part Number"
 	1    5200 5100
 	0    -1   -1   0
@@
 F 2 "Capacitor_SMD:C_0402_1005Metric_Pad0.74x0.62mm_HandSolder" H 3138 5350 50  0001 C CNN
 F 3 "https://www.digikey.com/en/products/detail/murata-electronics/GRM1555C1H3R0CA01D/3175191?s=N4IgTCBcDaIOICUCyBGArBgwigEgZgQAZMBBQlAERAF0BfIA" H 3100 5500 50  0001 C CNN
+F 4 "490-5872-1-ND" H 3100 5500 50  0001 C CNN "Digikey Part Number"
 	1    3100 5500
 	1    0    0    -1
@@
 F 2 "Inductor_SMD:L_0402_1005Metric_Pad0.77x0.64mm_HandSolder" H 3400 5300 50  0001 C CNN
 F 3 "https://www.digikey.com/en/products/detail/murata-electronics/LQG15HS10NJ02D/662872?s=N4IgTCBcDaIDIEUDiBGArACQMooAwDkApXMAERAF0BfIA" H 3400 5300 50  0001 C CNN
+F 4 "490-2623-1-ND" H 3400 5300 50  0001 C CNN "Digikey Part Number"
 	1    3400 5300
 	0    -1   -1   0
@@
 F 2 "Capacitor_SMD:C_0402_1005Metric_Pad0.74x0.62mm_HandSolder" H 2538 4950 50  0001 C CNN
 F 3 "https://www.digikey.com/en/products/detail/murata-electronics/GRM1555C1H1R2BA01D/3693934?s=N4IgTCBcDaIOICUCyBGArBgwigEihYAQgIIAMKAIiALoC%2BQA" H 2500 5100 50  0001 C CNN
+F 4 "490-6209-1-ND" H 2500 5100 50  0001 C CNN "Digikey Part Number"
 	1    2500 5100
 	1    0    0    -1
@@
 F 2 "Inductor_SMD:L_0402_1005Metric_Pad0.77x0.64mm_HandSolder" H 2850 5100 50  0001 C CNN
 F 3 "https://www.digikey.com/en/products/detail/murata-electronics/LQG15HS22NJ02D/662876?s=N4IgTCBcDaIDIEUDiBGArACQMpjAOQCkAGMAERAF0BfIA" H 2850 5100 50  0001 C CNN
+F 4 "490-2627-1-ND" H 2850 5100 50  0001 C CNN "Digikey Part Number"
 	1    2850 5100
 	1    0    0    -1
@@
 F 2 "Capacitor_SMD:C_0402_1005Metric_Pad0.74x0.62mm_HandSolder" H 2888 2850 50  0001 C CNN
 F 3 "https://www.digikey.com/en/products/detail/murata-electronics/GRM1555C1H1R1BA01D/3693932?s=N4IgTCBcDaIOICUCyBGArBgwigEihKAQgIIAMKAIiALoC%2BQA" H 2850 3000 50  0001 C CNN
+F 4 "490-8189-1-ND" H 2850 3000 50  0001 C CNN "Digikey Part Number"
 	1    2850 3000
 	0    -1   -1   0
@@
 F 2 "Connector_Coaxial:SMA_Amphenol_132134-16_Vertical" H 7800 3000 50  0001 C CNN
 F 3 "https://www.digikey.com/en/products/detail/amphenol-rf/132134/1011907" H 7800 3000 50  0001 C CNN
+F 4 "ACX1230-ND" H 7800 3450 50  0001 C CNN "Digikey Part Number"
 	1    7800 3450
 	1    0    0    -1
@@
 F 2 "Capacitor_SMD:C_0402_1005Metric_Pad0.74x0.62mm_HandSolder" H 5138 3050 50  0001 C CNN
 F 3 "https://www.digikey.com/en/products/detail/murata-electronics/GRM1555C1H120JA01D/3693831?s=N4IgTCBcDaIOICUCyBGArBgwigEisADAFICCBKAIiALoC%2BQA" H 5100 3200 50  0001 C CNN
+F 4 "490-5924-1-ND" H 5100 3200 50  0001 C CNN "Digikey Part Number"
 	1    5100 3200
 	0    -1   -1   0
@@
 F 2 "Capacitor_SMD:C_0402_1005Metric_Pad0.74x0.62mm_HandSolder" H 4588 3350 50  0001 C CNN
 F 3 "~" H 4550 3500 50  0001 C CNN
+F 4 "490-5939-1-ND" H 4550 3500 50  0001 C CNN "Digikey Part Number"
 	1    4550 3500
 	1    0    0    -1
@@
 F 2 "Capacitor_SMD:C_0402_1005Metric_Pad0.74x0.62mm_HandSolder" H 3738 3350 50  0001 C CNN
 F 3 "https://www.digikey.com/en/products/detail/avx-corporation/04025A1R0BAT2A/1116357" H 3700 3500 50  0001 C CNN
+F 4 "478-3659-1-ND" H 3700 3500 50  0001 C CNN "Digikey Part Number"
 	1    3700 3500
 	1    0    0    -1
@@
 F 2 "Capacitor_SMD:C_0402_1005Metric_Pad0.74x0.62mm_HandSolder" H 2538 2150 50  0001 C CNN
 F 3 "https://www.digikey.com/en/products/detail/murata-electronics/GRM1555C1H120JA01D/3693831?s=N4IgTCBcDaIOICUCyBGArBgwigEisADAFICCBKAIiALoC%2BQA" H 2500 2300 50  0001 C CNN
+F 4 "490-5924-1-ND" H 2500 2300 50  0001 C CNN "Digikey Part Number"
 	1    2500 2300
 	1    0    0    -1
@@
 F 2 "Capacitor_SMD:C_0402_1005Metric_Pad0.74x0.62mm_HandSolder" H 2538 3600 50  0001 C CNN
 F 3 "https://www.digikey.com/en/products/detail/murata-electronics/GRM1555C1H1R1BA01D/3693932?s=N4IgTCBcDaIOICUCyBGArBgwigEihKAQgIIAMKAIiALoC%2BQA" H 2500 3750 50  0001 C CNN
+F 4 "490-8189-1-ND" H 2500 3750 50  0001 C CNN "Digikey Part Number"
 	1    2500 3750
 	1    0    0    -1
@@
 F 2 "Inductor_SMD:L_0402_1005Metric_Pad0.77x0.64mm_HandSolder" H 3350 3200 50  0001 C CNN
 F 3 "https://www.digikey.com/en/products/detail/murata-electronics/LQG15HS2N0S02D/1795312?s=N4IgTCBcDaIDIEUDiBGArACQMpgHIAYt8wAREAXQF8g" H 3350 3200 50  0001 C CNN
+F 4 "490-6569-1-ND" H 3350 3200 50  0001 C CNN "Digikey Part Number"
 	1    3350 3200
 	0    -1   -1   0
@@
 F 2 "Inductor_SMD:L_0402_1005Metric_Pad0.77x0.64mm_HandSolder" H 4050 3200 50  0001 C CNN
 F 3 "https://www.digikey.com/en/products/detail/murata-electronics/LQG15HS2N0S02D/1795312?s=N4IgTCBcDaIDIEUDiBGArACQMpgHIAYt8wAREAXQF8g" H 4050 3200 50  0001 C CNN
+F 4 "490-6569-1-ND" H 4050 3200 50  0001 C CNN "Digikey Part Number"
 	1    4050 3200
 	0    -1   -1   0
@@
 F 2 "Inductor_SMD:L_0402_1005Metric_Pad0.77x0.64mm_HandSolder" H 2500 2700 50  0001 C CNN
 F 3 "https://www.digikey.com/en/products/detail/murata-electronics/LQG15HS2N4S02D/2594219?s=N4IgTCBcDaIDIEUDiBGArACQMpgHIBYsAGMAERAF0BfIA" H 2500 2700 50  0001 C CNN
+F 4 "490-8389-1-ND" H 2500 2700 50  0001 C CNN "Digikey Part Number"
 	1    2500 2700
 	1    0    0    -1
@@
 F 2 "Inductor_SMD:L_0402_1005Metric_Pad0.77x0.64mm_HandSolder" H 2900 3500 50  0001 C CNN
 F 3 "https://www.digikey.com/en/products/detail/murata-electronics/LQG15HS2N4S02D/2594219?s=N4IgTCBcDaIDIEUDiBGArACQMpgHIBYsAGMAERAF0BfIA" H 2900 3500 50  0001 C CNN
+F 4 "490-8389-1-ND" H 2900 3500 50  0001 C CNN "Digikey Part Number"
 	1    2900 3500
 	0    -1   -1   0
@@
 F 2 "Inductor_SMD:L_0402_1005Metric_Pad0.77x0.64mm_HandSolder" H 2300 3250 50  0001 C CNN
 F 3 "https://www.digikey.com/en/products/detail/murata-electronics/LQG15HS15NJ02D/662874?s=N4IgTCBcDaIDIEUDiBGArACQMroHICkAGMAERAF0BfIA" H 2300 3250 50  0001 C CNN
+F 4 "490-2625-1-ND" H 2300 3250 50  0001 C CNN "Digikey Part Number"
 	1    2300 3250
 	1    0    0    -1
@@
 F 2 "zigbeeCape:DPX252690DT-5032B1" H 6200 4150 50  0001 C CNN
 F 3 "https://www.digikey.com/en/products/detail/tdk-corporation/DPX252690DT-5032B1/5819342" H 6200 4150 50  0001 C CNN
+F 4 "445-174204-1-ND" H 6300 4150 50  0001 C CNN "Digikey Part Number"
 	1    6300 4150
 	1    0    0    -1
@@
 F 2 "Capacitor_SMD:C_0402_1005Metric_Pad0.74x0.62mm_HandSolder" H 7188 3800 50  0001 C CNN
 F 3 "https://www.digikey.com/en/products/detail/murata-electronics/GRM1555C1H101JA01D/3693829?s=N4IgTCBcDaIOICUCyBGArBgwigEigDCgFICChAIiALoC%2BQA" H 7150 3950 50  0001 C CNN
+F 4 "490-5922-1-ND" H 7150 3950 50  0001 C CNN "Digikey Part Number"
 	1    7150 3950
 	-1   0    0    1
