File: hardware/hardware/SwitchBoard/SwitchBoard/SwitchBoard.kicad_pcb (KiCad board)
At the start: 2 copper layers, 63.5 x 54.6 mm, 36 parts, among them SW1 SW_SPDT, SW2 SW_SPDT, SW3 SW_SPDT, SW4 SW_SPDT, SW5 SW_SPDT, SW6 SW_SPDT, SW7 SW_SPDT, SW8 SW_SPDT, U1 BeagleBone_P8, U2 MCP23S08, U3 BeagleBone_P9, U4 NCP1117-3.3_SOT223

Commit message: More progress on switchboard
Parts:
- C1, C2, C3, C4, R1, R2, U2, U4: moved to F.Cu
- moved C2 77.9 mm to (25.3, -43.3), turned to 90 degrees
- moved R2 73.4 mm to (25.7, -25.8), turned to 270 degrees
- moved C1 65.4 mm to (25.3, -39.6), turned to 90 degrees
- moved C3 60.8 mm to (32.0, -35.7), turned to 90 degrees
- moved R1 60.6 mm to (25.7, -29.3), turned to 90 degrees
- moved C4 55.3 mm to (34.4, -35.7), turned to 90 degrees
- moved U4 31.4 mm to (31.1, -41.3)
- moved D9 30.6 mm to (27.7, -14.0)
- moved R11 30.6 mm to (25.7, -14.0)
- moved U2 23.9 mm to (32.8, -27.7)
- moved R8 4.81 mm to (38.6, -37.3)
- moved R6 4.44 mm to (38.4, -17.5), turned to 0 degrees
- moved D4 1.15 mm to (37.7, -19.7)
- moved D6 1.02 mm to (37.7, -35.3)
- turned R4 to 270 degrees
Connections:
- U2 pad 12: SW_3 -> SW_5
- U2 pad 13: SW_4 -> SW_6
- U2 pad 14: SW_5 -> SW_7
- U2 pad 15: SW_6 -> SW_8
- U2 pad 16: SW_7 -> SW_3
- U2 pad 17: SW_8 -> SW_4
- U3 pad 22: CLK -> SCK
Routing:
- net GND: track 0.00 -> 51.7 mm, vias 0 -> 31
- net +3V3: track 0.00 -> 42.7 mm, vias 0 -> 22
- net SW_8: track 0.00 -> 41.5 mm
- net SW_5: track 0.00 -> 38.0 mm
- net SW_7: track 0.00 -> 34.7 mm
- net MOSI: track 0.00 -> 31.1 mm
- net MISO: track 0.00 -> 30.6 mm
- net SCK: track 0.00 -> 29.8 mm
- net SW_6: track 0.00 -> 29.0 mm
- net SW_4: track 0.00 -> 26.1 mm, vias 0 -> 2
- net SW_1: track 0.00 -> 24.5 mm
- net SW_3: track 0.00 -> 18.2 mm
- net SW_2: track 0.00 -> 16.4 mm
- net VDD: track 0.00 -> 6.52 mm, vias 0 -> 2
- net Net-(R2-Pad1): track 0.00 -> 2.87 mm
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Other:
- outline, holes or cut-outs redrawn

Commit message: Finished Layout with exception of power input
Parts:
- moved D9 7.08 mm to (34.5, -12.2)
- moved R11 6.84 mm to (32.3, -12.2)
- moved C1 4.04 mm to (28.1, -36.7), turned to 180 degrees
- moved C2 0.90 mm to (25.4, -42.4)
Routing:
- net ~CS: track 0.00 -> 26.6 mm, vias 0 -> 1
- net GND: track 51.7 -> 65.5 mm, vias 31 -> 28
- net +3V3: track 42.7 -> 47.5 mm, vias 22 -> 10
- net MOSI: track 31.1 -> 33.3 mm, vias 0 -> 1
- net VDD: track 6.52 -> 4.77 mm, vias 2 -> 1
- net SCK: track 29.8 -> 30.5 mm, vias 0 -> 1
- net MISO: track 30.6 -> 30.9 mm, vias 0 -> 1
- added copper zone on F.Cu, net +3V3
- added copper zone on B.Cu, net GND

Commit message: More switchboard updates
Parts:
- added J1: USB_B_Micro, microusb:UJ2-MIBH2-4-SMT-TR, F.Cu at (25.4, -15.5)
- added R12: DNP, Resistor_SMD:R_0603_1608Metric_Pad0.98x0.95mm_HandSolder, F.Cu at (29.7, -8.26)
- added R13: DNP, Resistor_SMD:R_0603_1608Metric_Pad0.98x0.95mm_HandSolder, F.Cu at (24.6, -8.26)
- added R14: 0, Resistor_SMD:R_0603_1608Metric_Pad0.98x0.95mm_HandSolder, F.Cu at (26.9, -8.26)
- moved R11 3.00 mm to (34.7, -14.0)
- moved D9 2.08 mm to (36.2, -10.9)
Connections:
- U3 pad 17: ~CS -> Net-(R14-Pad2)
Routing:
- net VDD: track 4.77 -> 30.7 mm, vias 1 -> 2
- net Net-(R12-Pad2): track 0.00 -> 12.0 mm
- net Net-(R13-Pad2): track 0.00 -> 6.70 mm
- net Net-(R14-Pad2): track 0.00 -> 6.59 mm
- net +3V3: track 47.5 -> 42.3 mm
- net ~CS: track 26.6 -> 23.8 mm, vias 1 -> 0
- net Net-(D9-Pad1): track 2.30 -> 0.00 mm
- net SCK: track 30.5 -> 30.2 mm, vias 1 -> 0

Commit message: Switchboardrev1 Complete
Parts:
- removed R13: DNP, Resistor_SMD:R_0603_1608Metric_Pad0.98x0.95mm_HandSolder
- added G***: LOGO, Graphics:bone1, F.Cu at (31.7, -42.6)
- moved C2 33.6 mm to (32.6, -9.55), turned to 270 degrees
- moved C1 27.3 mm to (24.6, -9.65), turned to 270 degrees
- moved U4 26.2 mm to (29.4, -15.1)
- moved J1 26.1 mm to (25.5, -41.6)
- moved D9 1.68 mm to (34.6, -10.3), turned to 270 degrees
- moved R12 0.91 mm to (30.6, -8.23)
- moved R14 0.16 mm to (26.8, -8.38)
Routing:
- net +3V3: track 42.3 -> 177.2 mm, vias 10 -> 18
- net VDD: track 30.7 -> 38.7 mm, vias 2 -> 0
- net Net-(R13-Pad2): track 6.70 -> 0.00 mm
- net Net-(R12-Pad2): track 12.0 -> 7.32 mm
- net GND: track 65.8 -> 69.0 mm, vias 28 -> 32
- net MOSI: track 33.4 -> 35.9 mm, vias 1 -> 0
- net Net-(D9-Pad1): track 0.00 -> 1.93 mm
- net ~CS: track 23.8 -> 22.0 mm, vias 0 -> 2
- net SW_4: track 26.1 -> 27.3 mm
- net SW_3: track 18.2 -> 17.3 mm
- net MISO: track 30.8 -> 31.3 mm, vias 1 -> 0
- removed copper zone on F.Cu, net +3V3
Other:
- board text added: "1"
- board text added: "2"
- board text added: "45"
- board text added: "46"
- board text added: "Iowa State CPR E/EE Senior Design Group 7 December 2021"
- board text added: "P8"
- board text added: "P9"
- board text added: "REV 1"
- board text added: "ZigBee Cape SwitchBoard"

Commit message: Finished Capev2 and switchv1
Parts:
- added R15: 10k, Resistor_SMD:R_0603_1608Metric_Pad0.98x0.95mm_HandSolder, F.Cu at (25.7, -23.3)
- moved R2 1.04 mm to (25.7, -26.8)
- moved R1 0.99 mm to (25.7, -30.3)
- moved G*** 0.37 mm to (31.3, -42.7), turned to 90 degrees
Connections:
- U2 pad 6: ~RESET -> Net-(R15-Pad1)
- U3 pad 18: MOSI -> MISO
- U3 pad 21: MISO -> MOSI
Routing:
- net Net-(R15-Pad1): track 0.00 -> 3.49 mm
- net MOSI: track 35.9 -> 32.4 mm
- net MISO: track 31.3 -> 33.8 mm
- net GND: track 69.0 -> 70.0 mm
