File: hardware/hardware/SwitchBoard/SwitchBoard/SwitchBoard.sch (KiCad schematic (older format))
At the start: 32 parts

Commit message: Finished Switchboard schematic and BOM
Parts:
- added C3: 1uF, symbol Device:C
- added C4: 10uF, symbol Device:C
- added D9: RED, symbol Device:LED
- added J1: USB_B_Micro, symbol Connector:USB_B_Micro
- added R11: 100, symbol Device:R
- C1, C2: renamed from C?; value C -> 10uF; Digikey Part Number (none) -> 1276-1038-1-ND
- D1, D2, D3, D4, D5, D6, D7, D8: renamed from D?; value LED -> RED; Digikey Part Number (none) -> 732-4978-1-ND
- R1, R2: renamed from R?; Digikey Part Number (none) -> 13-RT0603FRE1310KLCT-ND
- R10, R3, R4, R5, R6, R7, R8, R9: renamed from R?; Digikey Part Number (none) -> 118-CR0603AFX-1000ELFCT-ND
- SW1, SW2, SW3, SW4, SW5, SW6, SW7, SW8: renamed from SW?; Digikey Part Number (none) -> 401-2002-1-ND
- U1: renamed from U?; Digikey Part Number (none) -> 1528-1365-ND
- U2: renamed from U?; Digikey Part Number (none) -> MCP23S08-E/SO-ND
- U3: renamed from U?; Digikey Part Number (none) -> NA
- U4: renamed from U?; Digikey Part Number (none) -> 488-NCP1117IST33T3GCT-ND
Connections:
- net +3V3: now also C3.1, C4.1, D9.2 (A)
- net GND: now also C3.2, C4.2, J1.5 (GND), R11.2
- net VDD: now also J1.1 (VBUS)
- new net: D9.1 (K), R11.1
- no-connect marks 79 -> 83
Other:
- note added: "Do I need ESD protection and what should I use"
- moved on the sheet: R1, R2, U1, U2

Commit message: Finished schematic, BOM and started layout
Parts:
- removed J1: USB_B_Micro, symbol Connector:USB_B_Micro
- C1, C2, C3, C4: footprint (none) -> Capacitor_SMD:C_0603_1608Metric_Pad1.08x0.95mm_HandSolder
- D1, D2, D3, D4, D5, D6, D7, D8, D9: footprint (none) -> Diode_SMD:D_0603_1608Metric_Pad1.05x0.95mm_HandSolder
- R1, R10, R11, R2, R3, R4, R5, R6, R7, R8, R9: footprint (none) -> Resistor_SMD:R_0603_1608Metric_Pad0.98x0.95mm_HandSolder
- SW1, SW2, SW3, SW4, SW5, SW6, SW7, SW8: footprint (none) -> DPDT_Switch:DPDT
- U1, U3: footprint (none) -> Connector_PinHeader_2.54mm:PinHeader_2x23_P2.54mm_Vertical
- U2: footprint (none) -> Package_SO:SOIC-18W_7.5x11.6mm_P1.27mm
Connections:
- no-connect marks 83 -> 79

Commit message: More progress on switchboard
Connections:
- net CLK is gone; now on net SCK: U3.22 (SPIO_SCLK)
- net SW_3: now also U2.16 (GPIO6); no longer U2.12 (GPIO2)
- net SW_4: now also U2.17 (GPIO7); no longer U2.13 (GPIO3)
- net SW_5: now also U2.12 (GPIO2); no longer U2.14 (GPIO4)
- net SW_6: now also U2.13 (GPIO3); no longer U2.15 (GPIO5)
- net SW_7: now also U2.14 (GPIO4); no longer U2.16 (GPIO6)
- net SW_8: now also U2.15 (GPIO5); no longer U2.17 (GPIO7)
Changed lines of the file:
@@
 Text GLabel 3300 1900 2    50   Input ~ 0
 SW_2
+Text GLabel 3300 2400 2    50   Input ~ 0
+SW_3
+Text GLabel 3300 2500 2    50   Input ~ 0
+SW_4
 Text GLabel 3300 2000 2    50   Input ~ 0
-SW_3
+SW_5
 Text GLabel 3300 2100 2    50   Input ~ 0
-SW_4
+SW_6
 Text GLabel 3300 2200 2    50   Input ~ 0
-SW_5
+SW_7
 Text GLabel 3300 2300 2    50   Input ~ 0
-SW_6
-Text GLabel 3300 2400 2    50   Input ~ 0
-SW_7
-Text GLabel 3300 2500 2    50   Input ~ 0
 SW_8
 Wire Wire Line
@@
 Wire Wire Line
 	3300 1900 3150 1900
-Wire Wire Line
-	3150 2000 3300 2000
-Wire Wire Line
-	3150 2100 3300 2100
-Wire Wire Line
-	3150 2200 3300 2200
-Wire Wire Line
-	3150 2300 3300 2300
-Wire Wire Line
-	3150 2400 3300 2400
-Wire Wire Line
-	3150 2500 3300 2500
 $Comp
 L Switch:SW_SPDT SW2
@@
 $EndComp
 Text GLabel 6000 6250 2    50   Output ~ 0
-CLK
+SCK
 Text GLabel 6000 6350 2    50   Input ~ 0
 MISO
@@
 	1550 1600 1550 1550
 Connection ~ 1550 1600
+Wire Wire Line
+	3300 2500 3150 2500
+Wire Wire Line
+	3300 2400 3150 2400
+Wire Wire Line
+	3300 2300 3150 2300
+Wire Wire Line
+	3300 2200 3150 2200
+Wire Wire Line
+	3150 2100 3300 2100
+Wire Wire Line
+	3150 2000 3300 2000
 $EndSCHEMATC

Commit message: More switchboard updates
Parts:
- added J1: USB_B_Micro, microusb:UJ2-MIBH2-4-SMT-TR, symbol Connector:USB_B_Micro
- added R12, R13: DNP, Resistor_SMD:R_0603_1608Metric_Pad0.98x0.95mm_HandSolder, symbol Device:R
- added R14: 0, Resistor_SMD:R_0603_1608Metric_Pad0.98x0.95mm_HandSolder, symbol Device:R
Connections:
- net GND: now also J1.5 (GND), J1.6 (Shield)
- net VDD: now also J1.1 (VBUS)
- net ~CS: now also R12.1, R13.1, R14.1; no longer U3.17 (SPIO_CS0)
- net at U3.15 (GPIO_48): now also R13.2
- net at U3.25 (GPIO_117): now also R12.2
- new net: R14.2, U3.17 (SPIO_CS0)
Other:
- note removed: "Do I need ESD protection and what should I use"
Changed lines of the file:
@@
 Text GLabel 6000 6450 2    50   Output ~ 0
 MOSI
-Text GLabel 6000 6600 2    50   Input ~ 0
+Text GLabel 6450 6550 2    50   Input ~ 0
 ~CS
 Wire Wire Line
@@
 Wire Wire Line
 	5800 6450 6000 6450
-Wire Wire Line
-	5800 6550 5900 6550
-Wire Wire Line
-	5900 6550 5900 6600
-Wire Wire Line
-	5900 6600 6000 6600
 $Comp
 L power:+3.3V #PWR05
@@
 NoConn ~ 5800 5600
 NoConn ~ 5800 5500
-NoConn ~ 5800 5350
 NoConn ~ 5800 5250
 NoConn ~ 4500 5450
@@
 NoConn ~ 5800 5050
 NoConn ~ 5800 4950
-NoConn ~ 5800 4850
-NoConn ~ 5800 4750
 NoConn ~ 3000 7400
 NoConn ~ 3000 7300
@@
 Wire Wire Line
 	9850 5150 9850 5250
-Text Notes 1600 4000 0    50   ~ 0
-Do I need ESD protection and what should I use
 $Comp
 L Device:C C4
@@
 Wire Wire Line
 	3150 2000 3300 2000
+$Comp
+L Connector:USB_B_Micro J1
+U 1 1 61859C21
+P 1900 4050
+F 0 "J1" H 1957 4517 50  0000 C CNN
+F 1 "USB_B_Micro" H 1957 4426 50  0000 C CNN
+F 2 "microusb:UJ2-MIBH2-4-SMT-TR" H 2050 4000 50  0001 C CNN
+F 3 "~" H 2050 4000 50  0001 C CNN
+F 4 "102-4007-1-ND" H 1900 4050 50  0001 C CNN "Digikey Part Number"
+	1    1900 4050
+	1    0    0    -1
+$EndComp
+$Comp
+L power:GND #PWR0101
+U 1 1 6185AF6A
+P 1800 4550
+F 0 "#PWR0101" H 1800 4300 50  0001 C CNN
+F 1 "GND" H 1805 4377 50  0000 C CNN
+F 2 "" H 1800 4550 50  0001 C CNN
+F 3 "" H 1800 4550 50  0001 C CNN
+	1    1800 4550
+	1    0    0    -1
+$EndComp
+Wire Wire Line
+	1800 4550 1800 4500
+Wire Wire Line
+	1900 4450 1900 4500
+Wire Wire Line
+	1900 4500 1800 4500
+Connection ~ 1800 4500
+Wire Wire Line
+	1800 4500 1800 4450
+Wire Wire Line
+	2200 3850 2400 3850
+Wire Wire Line
+	2400 3850 2400 3750
+NoConn ~ 2200 4050
+NoConn ~ 2200 4150
+NoConn ~ 2200 4250
+$Comp
+L power:VDD #PWR0102
+U 1 1 618A770D
+P 2400 3750
+F 0 "#PWR0102" H 2400 3600 50  0001 C CNN
+F 1 "VDD" H 2415 3923 50  0000 C CNN
+F 2 "" H 2400 3750 50  0001 C CNN
+F 3 "" H 2400 3750 50  0001 C CNN
+	1    2400 3750
+	1    0    0    -1
+$EndComp
+$Comp
+L Device:R R12
+U 1 1 618B1AC7
+P 6100 5350
+F 0 "R12" V 5900 5350 50  0000 C CNN
+F 1 "DNP" V 6000 5350 50  0000 C CNN
+F 2 "Resistor_SMD:R_0603_1608Metric_Pad0.98x0.95mm_HandSolder" V 6030 5350 50  0001 C CNN
+F 3 "~" H 6100 5350 50  0001 C CNN
+	1    6100 5350
+	0    1    1    0
+$EndComp
+$Comp
+L Device:R R13
+U 1 1 618B2F48
+P 6100 4850
+F 0 "R13" V 6300 4850 50  0000 C CNN
+F 1 "DNP" V 6200 4850 50  0000 C CNN
+F 2 "Resistor_SMD:R_0603_1608Metric_Pad0.98x0.95mm_HandSolder" V 6030 4850 50  0001 C CNN
+F 3 "~" H 6100 4850 50  0001 C CNN
+	1    6100 4850
+	0    1    1    0
+$EndComp
+$Comp
+L Device:R R14
+U 1 1 618B99F0
+P 6100 6550
+F 0 "R14" V 6300 6550 50  0000 C CNN
+F 1 "0" V 6200 6550 50  0000 C CNN
+F 2 "Resistor_SMD:R_0603_1608Metric_Pad0.98x0.95mm_HandSolder" V 6030 6550 50  0001 C CNN
+F 3 "~" H 6100 6550 50  0001 C CNN
+	1    6100 6550
+	0    1    1    0
+$EndComp
+Wire Wire Line
+	5800 6550 5950 6550
+Wire Wire Line
+	6450 6550 6350 6550
+Wire Wire Line
+	6250 4850 6350 4850
+Wire Wire Line
+	6350 4850 6350 5350
+Connection ~ 6350 6550
+Wire Wire Line
+	6350 6550 6250 6550
+Wire Wire Line
+	5950 4850 5800 4850
+Wire Wire Line
+	5800 5350 5950 5350
+Wire Wire Line
+	6250 5350 6350 5350
+Connection ~ 6350 5350
+Wire Wire Line
+	6350 5350 6350 6550
 $EndSCHEMATC

Commit message: Switchboardrev1 Complete
Parts:
- R1, R2: Digikey Part Number 13-RT0603FRE1310KLCT-ND -> RMCF0603FT10K0CT-ND
- R14: Digikey Part Number (none) -> 541-0.0GCT-ND
Connections:
- net MISO: now also U3.18 (SPI0_D1); no longer U3.21 (SPIO_D0)
- net MOSI: now also U3.21 (SPIO_D0); no longer U3.18 (SPI0_D1)
Changed lines of the file:
@@
 F 2 "Resistor_SMD:R_0603_1608Metric_Pad0.98x0.95mm_HandSolder" V 1930 2800 50  0001 C CNN
 F 3 "~" H 2000 2800 50  0001 C CNN
-F 4 "13-RT0603FRE1310KLCT-ND" H 2000 2800 50  0001 C CNN "Digikey Part Number"
+F 4 "RMCF0603FT10K0CT-ND" H 2000 2800 50  0001 C CNN "Digikey Part Number"
 	1    2000 2800
 	1    0    0    -1
@@
 F 2 "Resistor_SMD:R_0603_1608Metric_Pad0.98x0.95mm_HandSolder" V 1630 2800 50  0001 C CNN
 F 3 "~" H 1700 2800 50  0001 C CNN
-F 4 "13-RT0603FRE1310KLCT-ND" H 1700 2800 50  0001 C CNN "Digikey Part Number"
+F 4 "RMCF0603FT10K0CT-ND" H 1700 2800 50  0001 C CNN "Digikey Part Number"
 	1    1700 2800
 	1    0    0    -1
@@
 SCK
 Text GLabel 6000 6350 2    50   Input ~ 0
+MOSI
+Text GLabel 6000 6450 2    50   Output ~ 0
 MISO
-Text GLabel 6000 6450 2    50   Output ~ 0
-MOSI
 Text GLabel 6450 6550 2    50   Input ~ 0
 ~CS
@@
 F 2 "Resistor_SMD:R_0603_1608Metric_Pad0.98x0.95mm_HandSolder" V 6030 6550 50  0001 C CNN
 F 3 "~" H 6100 6550 50  0001 C CNN
+F 4 "541-0.0GCT-ND" H 6100 6550 50  0001 C CNN "Digikey Part Number"
 	1    6100 6550
 	0    1    1    0

Commit message: Finished Capev2 and switchv1
Parts:
- removed R13: DNP, Resistor_SMD:R_0603_1608Metric_Pad0.98x0.95mm_HandSolder, symbol Device:R
- added R15: 10k, Resistor_SMD:R_0603_1608Metric_Pad0.98x0.95mm_HandSolder, symbol Device:R
Connections:
- net GND: now also R15.2
- net ~RESET: no longer names the net of U2.6 (~RESET)
- net ~RESET: now also R15.1
- no-connect marks 79 -> 81
Changed lines of the file:
@@
 L power:GND #PWR02
 U 1 1 6164DD9C
-P 1700 3250
-F 0 "#PWR02" H 1700 3000 50  0001 C CNN
-F 1 "GND" H 1705 3077 50  0000 C CNN
-F 2 "" H 1700 3250 50  0001 C CNN
-F 3 "" H 1700 3250 50  0001 C CNN
-	1    1700 3250
-	1    0    0    -1
-$EndComp
-Text GLabel 1350 2600 0    50   Input ~ 0
-~RESET
+P 1400 3250
+F 0 "#PWR02" H 1400 3000 50  0001 C CNN
+F 1 "GND" H 1405 3077 50  0000 C CNN
+F 2 "" H 1400 3250 50  0001 C CNN
+F 3 "" H 1400 3250 50  0001 C CNN
+	1    1400 3250
+	1    0    0    -1
+$EndComp
 $Comp
 L Device:R R2
@@
 $EndComp
 Wire Wire Line
-	2300 2600 1350 2600
-Wire Wire Line
 	2000 2650 2000 2500
 Wire Wire Line
@@
 	2000 3100 1700 3100
 Connection ~ 1700 3100
-Wire Wire Line
-	1700 3100 1700 3250
 Wire Wire Line
 	2300 2800 2250 2800
@@
 $EndComp
 $Comp
-L Device:R R13
-U 1 1 618B2F48
-P 6100 4850
-F 0 "R13" V 6300 4850 50  0000 C CNN
-F 1 "DNP" V 6200 4850 50  0000 C CNN
-F 2 "Resistor_SMD:R_0603_1608Metric_Pad0.98x0.95mm_HandSolder" V 6030 4850 50  0001 C CNN
-F 3 "~" H 6100 4850 50  0001 C CNN
-	1    6100 4850
-	0    1    1    0
-$EndComp
-$Comp
 L Device:R R14
 U 1 1 618B99F0
@@
 Wire Wire Line
 	6450 6550 6350 6550
-Wire Wire Line
-	6250 4850 6350 4850
-Wire Wire Line
-	6350 4850 6350 5350
 Connection ~ 6350 6550
 Wire Wire Line
 	6350 6550 6250 6550
 Wire Wire Line
-	5950 4850 5800 4850
-Wire Wire Line
 	5800 5350 5950 5350
 Wire Wire Line
 	6250 5350 6350 5350
-Connection ~ 6350 5350
 Wire Wire Line
 	6350 5350 6350 6550
+$Comp
+L Device:R R15
+U 1 1 618B728C
+P 1400 2800
+F 0 "R15" H 1470 2846 50  0000 L CNN
+F 1 "10k" H 1470 2755 50  0000 L CNN
+F 2 "Resistor_SMD:R_0603_1608Metric_Pad0.98x0.95mm_HandSolder" V 1330 2800 50  0001 C CNN
+F 3 "~" H 1400 2800 50  0001 C CNN
+F 4 "RMCF0603FT10K0CT-ND" H 1400 2800 50  0001 C CNN "Digikey Part Number"
+	1    1400 2800
+	1    0    0    -1
+$EndComp
+Wire Wire Line
+	1400 2650 1400 2600
+Wire Wire Line
+	1400 2600 2300 2600
+Wire Wire Line
+	1400 2950 1400 3100
+Wire Wire Line
+	1400 3100 1700 3100
+Wire Wire Line
+	1400 3250 1400 3100
+Connection ~ 1400 3100
+NoConn ~ 5800 4850
+NoConn ~ 5800 4750
 $EndSCHEMATC

Commit message: Finished and ordered boards
Parts:
- U4: Digikey Part Number 488-NCP1117IST33T3GCT-ND -> NCP1117ST33T3GOSCT-ND
Changed lines of the file:
@@
 F 1 "NCP1117-3.3_SOT223" H 8450 5251 50  0000 C CNN
 F 2 "Package_TO_SOT_SMD:SOT-223-3_TabPin2" H 8450 5300 50  0001 C CNN
-F 3 "http://www.onsemi.com/pub_link/Collateral/NCP1117-D.PDF" H 8550 4850 50  0001 C CNN
-F 4 "488-NCP1117IST33T3GCT-ND" H 8450 5100 50  0001 C CNN "Digikey Part Number"
+F 3 "" H 8550 4850 50  0001 C CNN
+F 4 "NCP1117ST33T3GOSCT-ND" H 8450 5100 50  0001 C CNN "Digikey Part Number"
 	1    8450 5100
 	1    0    0    -1
